File: dual_radio_addon.kicad_pcb (KiCad board)
At the start: 4 copper layers, 70 x 36 mm, 36 parts, among them J1 Mainboard, J2 Antenna switcher, J3 I2C, J4 I3C, U1 Module 1, U2 74LVC1GU04, U3 24C02BN, U4 Module 2, U5 74LVC1GU04, U6 Module 3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

Commit message: Fix connector orientation
Parts:
- added N1: OSHW, Symbol:OSHW-Logo2_9.8x8mm_SilkScreen, F.Cu at (-19.0, 10.5)
- J2: footprint Connector_PinHeader_2.54mm:PinHeader_2x05_P2.54mm_Vertical_SMD -> Connector_PinHeader_2.54mm:PinHeader_2x05_P2.54mm_Vertical
- moved J3 60.0 mm to (30.0, 8.00), turned to 90 degrees
- moved J4 60.0 mm to (-30.0, 8.00), turned to -90 degrees
- moved U3 30.5 mm to (14.5, 9.00), turned to 180 degrees
- moved J2 26.2 mm to (26.0, 15.2), turned to 180 degrees
- moved R10 24.5 mm to (6.00, 5.50), turned to 180 degrees
- moved C4 23.3 mm to (11.8, 12.2)
- moved JP1 20.4 mm to (9.42, 10.1), turned to -90 degrees
- moved R8 12.3 mm to (1.50, 5.50), turned to 180 degrees
- moved R2 5.37 mm to (-14.0, 5.50), turned to 0 degrees
- moved J1 3.81 mm to (-3.81, 12.0), turned to 90 degrees
- moved R5 3.08 mm to (-2.00, 5.50)
Connections:
- J1 pad 11: M1_BUSY -> M3_BUSY
- J1 pad 12: M1_DIO1 -> M3_DIO1
- J1 pad 14: M1_RESET -> M3_RESET
- J1 pad 18: M3_DIO1 -> M1_DIO1
- J1 pad 20: SPI_SCK -> SPI_MISO
- J1 pad 21: SPI_MISO -> SPI_SCK
- J1 pad 26: M3_BUSY -> M1_BUSY
- J1 pad 28: M3_RESET -> M1_RESET
- J2 pad 10: M3_RXEN -> M1_RXEN
- J2 pad 5: M1_TXEN -> M3_TXEN
- J2 pad 6: M1_RXEN -> M3_RXEN
- J2 pad 9: M3_TXEN -> M1_TXEN
Routing:
- net M3_NSS: track 33.0 -> 87.8 mm
- net M1_RXEN: track 42.1 -> 85.9 mm
- net M2_NSS: track 25.5 -> 66.2 mm
- net M1_TXEN: track 51.9 -> 86.2 mm
- net M3_BUSY: track 38.8 -> 15.8 mm
- net Net-(U6-BUSY): track 1.81 -> 24.6 mm
- net M2_TXEN: track 29.0 -> 49.8 mm, vias 0 -> 1
- net M3_RXEN: track 46.8 -> 26.2 mm, vias 0 -> 2
- net M2_RXEN: track 22.1 -> 41.5 mm, vias 0 -> 1
- net SPI_MOSI: track 66.2 -> 84.2 mm, vias 5 -> 4
- net +3.3V: track 64.3 -> 48.7 mm, vias 18 -> 21
- net SPI_SCK: track 69.8 -> 83.5 mm, vias 5 -> 4
- net M3_DIO1: track 41.1 -> 28.4 mm
- net M3_TXEN: track 39.9 -> 29.4 mm, vias 0 -> 2
- net GND: track 14.4 -> 4.26 mm, vias 111 -> 139
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Other:
- board text added: "<put funny artwork here>"
- board text added: "Ext. switch"
- board text added: "Tanmatsu"
