File: ebyte_addon.kicad_pcb (KiCad board)
At the start: 4 copper layers, 70 x 36 mm, 37 parts, among them J1 Mainboard, J2 Antenna switcher, J3 I2C, J4 I3C, U1 Module 1, U2 74LVC1GU04, U3 24C02BN, U4 Module 2, U5 74LVC1GU04, U6 Module 3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

Commit message: Rename files, add schematic and add notes to schematic
Other:
- board text removed: "<put funny artwork here>"
