File: ebyte_addon.kicad_sch (KiCad schematic)
At the start: 37 parts, among them J1 Mainboard, J2 Antenna switcher, J3 I2C, J4 I3C, U1 Module 1, U2 74LVC1GU04, U3 24C02BN, U4 Module 2, U5 74LVC1GU04, U6 Module 3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

Commit message: Rename files, add schematic and add notes to schematic
Other:
- note added: "Inverter on RX and TX enable is required for LoRa modules, on CC1101 modules the RX and TX enable pins are not connected, as a result the inverter may be left unnpopulated. This is why U2 and relating components are marked DNP."
- note added: "Left empty, user can solder in any of the supported modules"
- note added: "Populated with: CC1101 433MHz module"
- note added: "Populated with: LoRa 433MHz module"
Changed lines of the file:
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@@
 		(rev "0.1")
 		(company "Nicolai Electronics")
+		(comment 1 "License: CERN-OHL-P")
+		(comment 2 "Copyright © 2025 Nicolai Electronics")
+	)
+	(text "Inverter on RX and TX enable is required for\nLoRa modules, on CC1101 modules the RX and TX\nenable pins are not connected, as a result the\ninverter may be left unnpopulated. This is\nwhy U2 and relating components are marked DNP."
+		(exclude_from_sim no)
+		(at 231.394 16.764 0)
+		(effects
+			(font
+				(size 1.27 1.27)
+			)
+			(justify left top)
+		)
 	)
 	(text "Compatible with:\nE07-900M10S\nE07-400M10S\nE22-900M22S\nE22-400M22S"
@@
 		)
 	)
+	(text "Left empty, user can\nsolder in any of the\nsupported modules"
+		(exclude_from_sim no)
+		(at 91.694 179.07 0)
+		(effects
+			(font
+				(size 1.27 1.27)
+			)
+			(justify left top)
+		)
+	)
+	(text "Populated with:\nLoRa 433MHz module"
+		(exclude_from_sim no)
+		(at 91.948 120.904 0)
+		(effects
+			(font
+				(size 1.27 1.27)
+			)
+			(justify left top)
+		)
+	)
+	(text "Populated with:\nCC1101 433MHz module"
+		(exclude_from_sim no)
+		(at 91.44 62.484 0)
+		(effects
+			(font
+				(size 1.27 1.27)
+			)
+			(justify left top)
+		)
+	)
